File: kicad6/esp32-s3-darlington-array.kicad_pcb (KiCad board)
At the start: 2 copper layers, 46 x 31.5 mm, 31 parts, among them J1 B5B-XH-A, J2 USB_C_Receptacle_USB2.0, J3 Conn_01x03_Male, J4 Conn_01x08_Male, J5 Conn_01x03_Male, SW1 SW_Push, SW2 SW_Push, U1 ULN2003A, U2 ESP32-S3-WROOM-1, U3 AP2112K/RT9080-3.3

Commit message: Add schematics
Connections:
- net Net-(J1-Pad1) renamed /D13_Transistor
- net Net-(J1-Pad2) renamed /D12_Transistor
- net Net-(J1-Pad3) renamed /D11_Transistor
- net Net-(J1-Pad4) renamed /D10_Transistor
